Commit message: make changes in URDF to be compatible with UR3e

File: rh_p12_rn_a_description/urdf/rh_p12_rn_a.xacro (robot description, xacro)
@@ -1,4 +1,4 @@
 <?xml version="1.0"?>
-<robot name="rh_p12_rn_a" xmlns:xacro="http://www.ros.org/wiki/xacro">
+<robot xmlns:xacro="http://www.ros.org/wiki/xacro">
   <!-- some parameters -->
   <xacro:property name="pi" value="3.141592654" />
@@ -7,10 +7,8 @@
   <!-- Import Rviz colors -->
   <xacro:include filename="$(find rh_p12_rn_a_description)/urdf/materials.xacro" />
-  <!-- Used for fixing robot to Gazebo 'link 1' -->
-  <link name="world">
-  </link>
-  <joint name="world_fixed" type="fixed">
+  <!-- Used for fixing robot to the UR3e -->
+  <joint name="wrist_3_link_fixed" type="fixed">
     <origin xyz="0 0 0" rpy="0 0 0"/>
-    <parent link="world"/>
+    <parent link="wrist_3_link"/>
     <child link="rh_p12_rn_base"/>
   </joint>
@@ -49,8 +47,8 @@
     <type>transmission_interface/SimpleTransmission</type>
     <joint name="rh_p12_rn_a">
-      <hardwareInterface>hardware_interface/EffortJointInterface</hardwareInterface>
+      <hardwareInterface>hardware_interface/PositionJointInterface</hardwareInterface>
     </joint>
     <actuator name="motor_r1">
-      <hardwareInterface>hardware_interface/EffortJointInterface</hardwareInterface>
+      <hardwareInterface>hardware_interface/PositionJointInterface</hardwareInterface>
       <mechanicalReduction>1</mechanicalReduction>
     </actuator>
@@ -90,8 +88,8 @@
     <type>transmission_interface/SimpleTransmission</type>
     <joint name="rh_r2">
-      <hardwareInterface>hardware_interface/EffortJointInterface</hardwareInterface>
+      <hardwareInterface>hardware_interface/PositionJointInterface</hardwareInterface>
     </joint>
     <actuator name="motor_r2">
-      <hardwareInterface>hardware_interface/EffortJointInterface</hardwareInterface>
+      <hardwareInterface>hardware_interface/PositionJointInterface</hardwareInterface>
       <mechanicalReduction>1</mechanicalReduction>
     </actuator>
@@ -131,8 +129,8 @@
     <type>transmission_interface/SimpleTransmission</type>
     <joint name="rh_l1">
-      <hardwareInterface>hardware_interface/EffortJointInterface</hardwareInterface>
+      <hardwareInterface>hardware_interface/PositionJointInterface</hardwareInterface>
     </joint>
     <actuator name="motor_l1">
-      <hardwareInterface>hardware_interface/EffortJointInterface</hardwareInterface>
+      <hardwareInterface>hardware_interface/PositionJointInterface</hardwareInterface>
       <mechanicalReduction>1</mechanicalReduction>
     </actuator>
@@ -172,8 +170,8 @@
     <type>transmission_interface/SimpleTransmission</type>
     <joint name="rh_l2">
-      <hardwareInterface>hardware_interface/EffortJointInterface</hardwareInterface>
+      <hardwareInterface>hardware_interface/PositionJointInterface</hardwareInterface>
     </joint>
     <actuator name="motor_l2">
-      <hardwareInterface>hardware_interface/EffortJointInterface</hardwareInterface>
+      <hardwareInterface>hardware_interface/PositionJointInterface</hardwareInterface>
       <mechanicalReduction>1</mechanicalReduction>
     </actuator>

Commit message: rotate 90 degrees on gripper

File: rh_p12_rn_a_description/urdf/rh_p12_rn_a.xacro (robot description, xacro)
@@ -9,5 +9,5 @@
   <!-- Used for fixing robot to the UR3e -->
   <joint name="wrist_3_link_fixed" type="fixed">
-    <origin xyz="0 0 0" rpy="0 0 0"/>
+    <origin xyz="0 0 0" rpy="0 0 1.5707"/>
     <parent link="wrist_3_link"/>
     <child link="rh_p12_rn_base"/>

Commit message: mimic gripper joints in Gazebo based on a single gripper joint

File: rh_p12_rn_a_description/urdf/rh_p12_rn_a.xacro (robot description, xacro)
@@ -5,4 +5,5 @@
   <!-- Import all Gazebo-customization elements, including Gazebo colors -->
   <xacro:include filename="$(find rh_p12_rn_a_description)/urdf/rh_p12_rn_a.gazebo" />
+  <xacro:include filename="$(find rh_p12_rn_a_description)/urdf/inertia_tensors.urdf.xacro" />
   <!-- Import Rviz colors -->
   <xacro:include filename="$(find rh_p12_rn_a_description)/urdf/materials.xacro" />
@@ -34,4 +35,33 @@
       <inertia ixx="1.0" ixy="0.0" ixz="0.0" iyy="1.0" iyz="0.0" izz="1.0" />
     </inertial>
+  </link>
+  <!-- Finger Motor Joint -->
+  <joint name="gripper" type="revolute">
+    <origin xyz="0 0.0 0" rpy="0 0 0" />
+    <axis xyz="1 0 0" />
+    <limit lower="0" upper="1.15" effort="4" velocity="5" />
+    <parent link="rh_p12_rn_base" />
+    <child link="gripper_link" />
+  </joint>
+  <transmission name="gripper_transmission">
+    <type>transmission_interface/SimpleTransmission</type>
+    <joint name="gripper">
+      <hardwareInterface>hardware_interface/PositionJointInterface</hardwareInterface>
+    </joint>
+    <actuator name="gripper_motor">
+      <hardwareInterface>hardware_interface/PositionJointInterface</hardwareInterface>
+      <mechanicalReduction>1</mechanicalReduction>
+    </actuator>
+  </transmission>
+  <link name="gripper_link">
+    <!--<inertial>
+    <origin xyz="0 0 0" rpy="0 0 0" />
+    <mass value="0.01" />
+    <inertia ixx="1.0e-6" ixy="0.0" ixz="0.0" iyy="1.0e-6" iyz="0.0" izz="1.0e-6" />
+    </inertial>
+    -->
+    <xacro:inertial_cuboid_with_pose mass="0.01" x_length="0.04" y_length="0.04" z_length="0.04" >
+      <origin xyz="0.0 0.0 0.0" rpy="0 0 0" />
+    </xacro:inertial_cuboid_with_pose>
   </link>
   <!-- Joint -->
@@ -43,6 +73,17 @@
     <limit velocity="6.5" effort="1000" lower="0.0" upper="1.1" />
     <dynamics damping="0.7"/>
-  </joint>
-  <transmission name="tran_r1">
+    <mimic joint="gripper" multiplier="1" offset="0"/>
+  </joint>
+  <gazebo>
+    <plugin name="mimic_joint_rh_p12_rn_a" filename="libroboticsgroup_gazebo_mimic_joint_plugin.so">
+      <joint>gripper</joint>
+      <mimicJoint>rh_p12_rn_a</mimicJoint>
+      <multiplier>1</multiplier>
+      <offset>0</offset>
+      <maxEffort>4</maxEffort>
+      <hasPID/>
+    </plugin>
+  </gazebo>
+  <!--transmission name="tran_r1">
     <type>transmission_interface/SimpleTransmission</type>
     <joint name="rh_p12_rn_a">
@@ -53,5 +94,5 @@
       <mechanicalReduction>1</mechanicalReduction>
     </actuator>
-  </transmission>
+  </transmission-->
   <!-- rh_p12_rn_r1 -->
   <link name="rh_p12_rn_r1">
@@ -84,6 +125,17 @@
     <limit velocity="6.5" effort="1000" lower="0.0" upper="1.0" />
     <dynamics damping="0.7"/>
-  </joint>
-  <transmission name="tran_r2">
+    <mimic joint="gripper" multiplier="0.909" offset="0"/>
+  </joint>
+  <gazebo>
+    <plugin name="mimic_joint_rh_r2" filename="libroboticsgroup_gazebo_mimic_joint_plugin.so">
+      <joint>gripper</joint>
+      <mimicJoint>rh_r2</mimicJoint>
+      <multiplier>0.909</multiplier>
+      <offset>0</offset>
+      <maxEffort>4</maxEffort>
+      <hasPID/>
+    </plugin>
+  </gazebo>
+  <!--transmission name="tran_r2">
     <type>transmission_interface/SimpleTransmission</type>
     <joint name="rh_r2">
@@ -94,5 +146,5 @@
       <mechanicalReduction>1</mechanicalReduction>
     </actuator>
-  </transmission>
+  </transmission-->
   <!-- rh_p12_rn_r2 -->
   <link name="rh_p12_rn_r2">
@@ -125,6 +177,17 @@
     <limit velocity="6.5" effort="1000" lower="0.0" upper="1.1" />
     <dynamics damping="0.7"/>
-  </joint>
-  <transmission name="tran_l1">
+    <mimic joint="gripper" multiplier="1" offset="0"/>
+  </joint>
+  <gazebo>
+    <plugin name="mimic_joint_rh_l1" filename="libroboticsgroup_gazebo_mimic_joint_plugin.so">
+      <joint>gripper</joint>
+      <mimicJoint>rh_l1</mimicJoint>
+      <multiplier>1</multiplier>
+      <offset>0</offset>
+      <maxEffort>4</maxEffort>
+      <hasPID/>
+    </plugin>
+  </gazebo>
+  <!--transmission name="tran_l1">
     <type>transmission_interface/SimpleTransmission</type>
     <joint name="rh_l1">
@@ -135,5 +198,5 @@
       <mechanicalReduction>1</mechanicalReduction>
     </actuator>
-  </transmission>
+  </transmission-->
   <!-- rh_p12_rn_l1 -->
   <link name="rh_p12_rn_l1">
@@ -166,6 +229,17 @@
     <limit velocity="6.5" effort="1000" lower="0.0" upper="1.0" />
     <dynamics damping="0.7"/>
-  </joint>
-  <transmission name="tran_l2">
+    <mimic joint="gripper" multiplier="0.909" offset="0"/>
+  </joint>
+  <gazebo>
+    <plugin name="mimic_joint_rh_l2" filename="libroboticsgroup_gazebo_mimic_joint_plugin.so">
+      <joint>gripper</joint>
+      <mimicJoint>rh_l2</mimicJoint>
+      <multiplier>0.909</multiplier>
+      <offset>0</offset>
+      <maxEffort>4</maxEffort>
+      <hasPID/>
+    </plugin>
+  </gazebo>
+  <!--transmission name="tran_l2">
     <type>transmission_interface/SimpleTransmission</type>
     <joint name="rh_l2">
@@ -176,5 +250,5 @@
       <mechanicalReduction>1</mechanicalReduction>
     </actuator>
-  </transmission>
+  </transmission-->
   <!-- rh_p12_rn_l2 -->
   <link name="rh_p12_rn_l2">

Commit message: initial changes on xacro to make it work with ROS2

File: rh_p12_rn_a_description/urdf/rh_p12_rn_a.xacro (robot description, xacro)
@@ -1,15 +1,15 @@
 <?xml version="1.0"?>
-<robot xmlns:xacro="http://www.ros.org/wiki/xacro">
-  <!-- some parameters -->
-  <xacro:property name="pi" value="3.141592654" />
+<robot name="rh_p12_rn_a" xmlns:xacro="http://wiki.ros.org/xacro">
   <!-- Import all Gazebo-customization elements, including Gazebo colors -->
-  <xacro:include filename="$(find rh_p12_rn_a_description)/urdf/rh_p12_rn_a.gazebo" />
+  <!-- <xacro:include filename="$(find rh_p12_rn_a_description)/urdf/rh_p12_rn_a.gazebo" /> -->
   <xacro:include filename="$(find rh_p12_rn_a_description)/urdf/inertia_tensors.urdf.xacro" />
   <!-- Import Rviz colors -->
   <xacro:include filename="$(find rh_p12_rn_a_description)/urdf/materials.xacro" />
+  <!-- Global reference link -->
+  <link name="world"/>
   <!-- Used for fixing robot to the UR3e -->
-  <joint name="wrist_3_link_fixed" type="fixed">
+  <joint name="world_fixed" type="fixed">
     <origin xyz="0 0 0" rpy="0 0 1.5707"/>
-    <parent link="wrist_3_link"/>
+    <parent link="world"/>
     <child link="rh_p12_rn_base"/>
   </joint>
@@ -44,5 +44,5 @@
     <child link="gripper_link" />
   </joint>
-  <transmission name="gripper_transmission">
+  <!-- <transmission name="gripper_transmission">
     <type>transmission_interface/SimpleTransmission</type>
     <joint name="gripper">
@@ -53,5 +53,5 @@
       <mechanicalReduction>1</mechanicalReduction>
     </actuator>
-  </transmission>
+  </transmission> -->
   <link name="gripper_link">
     <!--<inertial>
