Commit message: update xacro to the new format from OM-Y

File: rh_p12_rn_a_description/urdf/rh_p12_rn_a.xacro (robot description, xacro)
@@ -1,23 +1,26 @@
 <?xml version="1.0"?>
-<robot name="rh_p12_rn_a" xmlns:xacro="http://wiki.ros.org/xacro">
-  <!-- Import all Gazebo-customization elements, including Gazebo colors -->
-  <!-- <xacro:include filename="$(find rh_p12_rn_a_description)/urdf/rh_p12_rn_a.gazebo" /> -->
-  <xacro:include filename="$(find rh_p12_rn_a_description)/urdf/inertia_tensors.urdf.xacro" />
-  <!-- Import Rviz colors -->
+<!-- rh_p12_rn_a gripper -->
+<robot name="rh_p12_rn_a" xmlns:xacro="http://www.ros.org/wiki/xacro">
+  <xacro:property name="prefix" default="" />
   <xacro:include filename="$(find rh_p12_rn_a_description)/urdf/materials.xacro" />
+  <xacro:include filename="$(find rh_p12_rn_a_description)/urdf/rh_p12_rn_a.gazebo" />
+  <xacro:include filename="$(find rh_p12_rn_a_description)/urdf/ros2_control.xacro" />
+  <xacro:property
+    name="meshes_file_direction"
+    value="package://rh_p12_rn_a_description/meshes"/>
   <!-- Global reference link -->
   <link name="world"/>
   <!-- Used for fixing robot to the UR3e -->
   <joint name="world_fixed" type="fixed">
-    <origin xyz="0 0 0" rpy="0 0 1.5707"/>
+    <origin xyz="0 0 0" rpy="0 0 0"/>
     <parent link="world"/>
-    <child link="rh_p12_rn_base"/>
+    <child link="${prefix}rh_p12_rn_base"/>
   </joint>
   <!-- base -->
-  <link name="rh_p12_rn_base">
+  <link name="${prefix}rh_p12_rn_base">
     <collision>
       <origin xyz="0 0 0" rpy="0 0 0"/>
       <geometry>
-        <mesh filename="package://rh_p12_rn_a_description/meshes/base.stl" scale="0.001 0.001 0.001"/>
+        <mesh filename="${meshes_file_direction}/base.stl" scale="0.001 0.001 0.001"/>
       </geometry>
     </collision>
@@ -25,80 +28,31 @@
       <origin xyz="0 0 0" rpy="0 0 0"/>
       <geometry>
-        <mesh filename="package://rh_p12_rn_a_description/meshes/base.stl" scale="0.001 0.001 0.001"/>
+        <mesh filename="${meshes_file_direction}/base.stl" scale="0.001 0.001 0.001"/>
       </geometry>
-      <material name="grey"/>
+              <material name="grey">
+        <color rgba="0.2 0.2 0.2 1"/>
+      </material>
     </visual>
     <inertial>
       <origin xyz="0.000 0.000 0.032" rpy="0 0 0"/>
       <mass value="0.236"/>
-      <!--<inertia ixx="0.00017" ixy="0.0" ixz="0.0" iyy="0.00011" iyz="0.0" izz="0.00017" />-->
-      <inertia ixx="1.0" ixy="0.0" ixz="0.0" iyy="1.0" iyz="0.0" izz="1.0" />
+      <inertia ixx="0.000001" ixy="0.0" ixz="0.0" iyy="0.000001" iyz="0.0" izz="0.000001" />
     </inertial>
   </link>
-  <!-- Finger Motor Joint -->
-  <joint name="gripper" type="revolute">
-    <origin xyz="0 0.0 0" rpy="0 0 0" />
-    <axis xyz="1 0 0" />
-    <limit lower="0" upper="1.15" effort="4" velocity="5" />
-    <parent link="rh_p12_rn_base" />
-    <child link="gripper_link" />
-  </joint>
-  <!-- <transmission name="gripper_transmission">
-    <type>transmission_interface/SimpleTransmission</type>
-    <joint name="gripper">
-      <hardwareInterface>hardware_interface/PositionJointInterface</hardwareInterface>
-    </joint>
-    <actuator name="gripper_motor">
-      <hardwareInterface>hardware_interface/PositionJointInterface</hardwareInterface>
-      <mechanicalReduction>1</mechanicalReduction>
-    </actuator>
-  </transmission> -->
-  <link name="gripper_link">
-    <!--<inertial>
-    <origin xyz="0 0 0" rpy="0 0 0" />
-    <mass value="0.01" />
-    <inertia ixx="1.0e-6" ixy="0.0" ixz="0.0" iyy="1.0e-6" iyz="0.0" izz="1.0e-6" />
-    </inertial>
-    -->
-    <xacro:inertial_cuboid_with_pose mass="0.01" x_length="0.04" y_length="0.04" z_length="0.04" >
-      <origin xyz="0.0 0.0 0.0" rpy="0 0 0" />
-    </xacro:inertial_cuboid_with_pose>
-  </link>
   <!-- Joint -->
-  <joint name="rh_p12_rn_a" type="revolute">
-    <parent link="rh_p12_rn_base"/>
-    <child link="rh_p12_rn_r1"/>
+  <joint name="${prefix}rh_r1_joint" type="revolute">
+    <parent link="${prefix}rh_p12_rn_base"/>
+    <child link="${prefix}rh_p12_rn_r1"/>
     <origin xyz="0.0 0.008 0.048" rpy="0 0 0"/>
     <axis xyz="1 0 0"/>
-    <limit velocity="6.5" effort="1000" lower="0.0" upper="1.1" />
+    <limit velocity="6.5" effort="1000" lower="-0.1" upper="1.1"/>
     <dynamics damping="0.7"/>
-    <mimic joint="gripper" multiplier="1" offset="0"/>
   </joint>
-  <gazebo>
-    <plugin name="mimic_joint_rh_p12_rn_a" filename="libroboticsgroup_gazebo_mimic_joint_plugin.so">
-      <joint>gripper</joint>
-      <mimicJoint>rh_p12_rn_a</mimicJoint>
-      <multiplier>1</multiplier>
-      <offset>0</offset>
-      <maxEffort>4</maxEffort>
-      <hasPID/>
-    </plugin>
-  </gazebo>
-  <!--transmission name="tran_r1">
-    <type>transmission_interface/SimpleTransmission</type>
-    <joint name="rh_p12_rn_a">
-      <hardwareInterface>hardware_interface/PositionJointInterface</hardwareInterface>
-    </joint>
-    <actuator name="motor_r1">
-      <hardwareInterface>hardware_interface/PositionJointInterface</hardwareInterface>
-      <mechanicalReduction>1</mechanicalReduction>
-    </actuator>
-  </transmission-->
   <!-- rh_p12_rn_r1 -->
-  <link name="rh_p12_rn_r1">
+  <link name="${prefix}rh_p12_rn_r1">
     <collision>
       <origin xyz="0 0 0" rpy="0 0 0"/>
       <geometry>
-        <mesh filename="package://rh_p12_rn_a_description/meshes/r1.stl" scale="0.001 0.001 0.001"/>
+        <mesh filename="${meshes_file_direction}/r1.stl" scale="0.001 0.001 0.001"/>
       </geometry>
     </collision>
@@ -106,51 +60,32 @@
       <origin xyz="0 0 0" rpy="0 0 0"/>
       <geometry>
-        <mesh filename="package://rh_p12_rn_a_description/meshes/r1.stl" scale="0.001 0.001 0.001"/>
+        <mesh filename="${meshes_file_direction}/r1.stl" scale="0.001 0.001 0.001"/>
       </geometry>
-      <material name="grey"/>
+              <material name="grey">
+        <color rgba="0.2 0.2 0.2 1"/>
+      </material>
     </visual>
     <inertial>
       <origin xyz="0.000 0.034 0.004" rpy="0 0 0"/>
       <mass value="0.068"/>
-      <!--<inertia ixx="0.00004" ixy="0.0" ixz="0.0" iyy="0.00002" iyz="-0.00001" izz="0.00002" />-->
-      <inertia ixx="1.0" ixy="0.0" ixz="0.0" iyy="1.0" iyz="0.0" izz="1.0" />
+      <inertia ixx="0.000001" ixy="0.0" ixz="0.0" iyy="0.000001" iyz="0.0" izz="0.000001" />
     </inertial>
   </link>
   <!-- Right Joint 2 -->
-  <joint name="rh_r2" type="revolute">
-    <parent link="rh_p12_rn_r1"/>
-    <child link="rh_p12_rn_r2"/>
+  <joint name="${prefix}rh_r2" type="revolute">
+    <parent link="${prefix}rh_p12_rn_r1"/>
+    <child link="${prefix}rh_p12_rn_r2"/>
     <origin xyz="0.0 0.0493634 0.0285" rpy="0 0 0"/>
     <axis xyz="-1 0 0"/>
     <limit velocity="6.5" effort="1000" lower="0.0" upper="1.0" />
     <dynamics damping="0.7"/>
-    <mimic joint="gripper" multiplier="0.909" offset="0"/>
+    <mimic joint="${prefix}rh_r1_joint" multiplier="1"/>
   </joint>
-  <gazebo>
-    <plugin name="mimic_joint_rh_r2" filename="libroboticsgroup_gazebo_mimic_joint_plugin.so">
-      <joint>gripper</joint>
-      <mimicJoint>rh_r2</mimicJoint>
-      <multiplier>0.909</multiplier>
-      <offset>0</offset>
-      <maxEffort>4</maxEffort>
-      <hasPID/>
-    </plugin>
-  </gazebo>
-  <!--transmission name="tran_r2">
-    <type>transmission_interface/SimpleTransmission</type>
-    <joint name="rh_r2">
-      <hardwareInterface>hardware_interface/PositionJointInterface</hardwareInterface>
-    </joint>
-    <actuator name="motor_r2">
-      <hardwareInterface>hardware_interface/PositionJointInterface</hardwareInterface>
-      <mechanicalReduction>1</mechanicalReduction>
-    </actuator>
-  </transmission-->
   <!-- rh_p12_rn_r2 -->
-  <link name="rh_p12_rn_r2">
+  <link name="${prefix}rh_p12_rn_r2">
     <collision>
       <origin xyz="0 0 0" rpy="0 0 0"/>
       <geometry>
-        <mesh filename="package://rh_p12_rn_a_description/meshes/r2.stl" scale="0.001 0.001 0.001"/>
+        <mesh filename="${meshes_file_direction}/r2.stl" scale="0.001 0.001 0.001"/>
       </geometry>
     </collision>
@@ -158,51 +93,32 @@
       <origin xyz="0 0 0" rpy="0 0 0"/>
       <geometry>
-        <mesh filename="package://rh_p12_rn_a_description/meshes/r2.stl" scale="0.001 0.001 0.001"/>
+        <mesh filename="${meshes_file_direction}/r2.stl" scale="0.001 0.001 0.001"/>
       </geometry>
-      <material name="grey"/>
+              <material name="grey">
+        <color rgba="0.2 0.2 0.2 1"/>
+      </material>
     </visual>
     <inertial>
       <origin xyz="0.000 0.006 0.011" rpy="0 0 0"/>
       <mass value="0.022"/>
-      <!--<inertia ixx="0.0" ixy="0.0" ixz="0.0" iyy="0.00001" iyz="0.0" izz="0.0" />-->
-      <inertia ixx="1.0" ixy="0.0" ixz="0.0" iyy="1.0" iyz="0.0" izz="1.0" />
+      <inertia ixx="0.000001" ixy="0.0" ixz="0.0" iyy="0.000001" iyz="0.0" izz="0.000001" />
     </inertial>
   </link>
   <!-- Left Joint 1 -->
-  <joint name="rh_l1" type="revolute">
-    <parent link="rh_p12_rn_base"/>
-    <child link="rh_p12_rn_l1"/>
+  <joint name="${prefix}rh_l1" type="revolute">
+    <parent link="${prefix}rh_p12_rn_base"/>
+    <child link="${prefix}rh_p12_rn_l1"/>
     <origin xyz="0.0 -0.008 0.048" rpy="0 0 0"/>
     <axis xyz="-1 0 0"/>
-    <limit velocity="6.5" effort="1000" lower="0.0" upper="1.1" />
+    <limit velocity="6.5" effort="1000" lower="-0.1" upper="1.1" />
     <dynamics damping="0.7"/>
-    <mimic joint="gripper" multiplier="1" offset="0"/>
+    <mimic joint="${prefix}rh_r1_joint" multiplier="1"/>
   </joint>
-  <gazebo>
-    <plugin name="mimic_joint_rh_l1" filename="libroboticsgroup_gazebo_mimic_joint_plugin.so">
-      <joint>gripper</joint>
-      <mimicJoint>rh_l1</mimicJoint>
-      <multiplier>1</multiplier>
-      <offset>0</offset>
-      <maxEffort>4</maxEffort>
-      <hasPID/>
-    </plugin>
-  </gazebo>
-  <!--transmission name="tran_l1">
-    <type>transmission_interface/SimpleTransmission</type>
-    <joint name="rh_l1">
-      <hardwareInterface>hardware_interface/PositionJointInterface</hardwareInterface>
-    </joint>
-    <actuator name="motor_l1">
-      <hardwareInterface>hardware_interface/PositionJointInterface</hardwareInterface>
-      <mechanicalReduction>1</mechanicalReduction>
-    </actuator>
-  </transmission-->
   <!-- rh_p12_rn_l1 -->
-  <link name="rh_p12_rn_l1">
+  <link name="${prefix}rh_p12_rn_l1">
     <collision>
       <origin xyz="0 0 0" rpy="0 0 0"/>
       <geometry>
-        <mesh filename="package://rh_p12_rn_a_description/meshes/l1.stl" scale="0.001 0.001 0.001"/>
+        <mesh filename="${meshes_file_direction}/l1.stl" scale="0.001 0.001 0.001"/>
       </geometry>
     </collision>
@@ -210,51 +126,32 @@
       <origin xyz="0 0 0" rpy="0 0 0"/>
       <geometry>
-        <mesh filename="package://rh_p12_rn_a_description/meshes/l1.stl" scale="0.001 0.001 0.001"/>
+        <mesh filename="${meshes_file_direction}/l1.stl" scale="0.001 0.001 0.001"/>
       </geometry>
-      <material name="grey"/>
+              <material name="grey">
+        <color rgba="0.2 0.2 0.2 1"/>
+      </material>
     </visual>
     <inertial>
       <origin xyz="0.000 -0.034 0.004" rpy="0 0 0"/>
       <mass value="0.068"/>
-      <!--<inertia ixx="0.00004" ixy="0.0" ixz="0.0" iyy="0.00002" iyz="0.00001" izz="0.00002" />-->
-      <inertia ixx="1.0" ixy="0.0" ixz="0.0" iyy="1.0" iyz="0.0" izz="1.0" />
+      <inertia ixx="0.000001" ixy="0.0" ixz="0.0" iyy="0.000001" iyz="0.0" izz="0.000001" />
     </inertial>
   </link>
   <!-- Left Joint 2 -->
-  <joint name="rh_l2" type="revolute">
-    <parent link="rh_p12_rn_l1"/>
-    <child link="rh_p12_rn_l2"/>
+  <joint name="${prefix}rh_l2" type="revolute">
+    <parent link="${prefix}rh_p12_rn_l1"/>
+    <child link="${prefix}rh_p12_rn_l2"/>
     <origin xyz="0.0 -0.0493634 0.0285" rpy="0 0 0"/>
     <axis xyz="1 0 0"/>
     <limit velocity="6.5" effort="1000" lower="0.0" upper="1.0" />
     <dynamics damping="0.7"/>
-    <mimic joint="gripper" multiplier="0.909" offset="0"/>
+    <mimic joint="${prefix}rh_r1_joint" multiplier="1"/>
   </joint>
-  <gazebo>
-    <plugin name="mimic_joint_rh_l2" filename="libroboticsgroup_gazebo_mimic_joint_plugin.so">
-      <joint>gripper</joint>
-      <mimicJoint>rh_l2</mimicJoint>
-      <multiplier>0.909</multiplier>
-      <offset>0</offset>
-      <maxEffort>4</maxEffort>
-      <hasPID/>
-    </plugin>
-  </gazebo>
-  <!--transmission name="tran_l2">
-    <type>transmission_interface/SimpleTransmission</type>
-    <joint name="rh_l2">
-      <hardwareInterface>hardware_interface/PositionJointInterface</hardwareInterface>
-    </joint>
-    <actuator name="motor_l2">
-      <hardwareInterface>hardware_interface/PositionJointInterface</hardwareInterface>
-      <mechanicalReduction>1</mechanicalReduction>
-    </actuator>
-  </transmission-->
   <!-- rh_p12_rn_l2 -->
-  <link name="rh_p12_rn_l2">
+  <link name="${prefix}rh_p12_rn_l2">
     <collision>
       <origin xyz="0 0 0" rpy="0 0 0"/>
       <geometry>
-        <mesh filename="package://rh_p12_rn_a_description/meshes/l2.stl" scale="0.001 0.001 0.001"/>
+        <mesh filename="${meshes_file_direction}/l2.stl" scale="0.001 0.001 0.001"/>
       </geometry>
     </collision>
@@ -262,23 +159,24 @@
       <origin xyz="0 0 0" rpy="0 0 0"/>
       <geometry>
-        <mesh filename="package://rh_p12_rn_a_description/meshes/l2.stl" scale="0.001 0.001 0.001"/>
+        <mesh filename="${meshes_file_direction}/l2.stl" scale="0.001 0.001 0.001"/>
       </geometry>
-      <material name="grey"/>
+              <material name="grey">
+        <color rgba="0.2 0.2 0.2 1"/>
+      </material>
     </visual>
     <inertial>
       <origin xyz="0.000 -0.006 0.011" rpy="0 0 0"/>
       <mass value="0.022"/>
-      <!--<inertia ixx="0.0" ixy="0.0" ixz="0.0" iyy="0.00001" iyz="0.0" izz="0.0" />-->
-      <inertia ixx="1.0" ixy="0.0" ixz="0.0" iyy="1.0" iyz="0.0" izz="1.0" />
+      <inertia ixx="0.000001" ixy="0.0" ixz="0.0" iyy="0.000001" iyz="0.0" izz="0.000001" />
     </inertial>
   </link>
   <!-- Gripper end effector joint -->
-  <joint name="rh_p12_rn_ee_joint" type="fixed">
+  <joint name="${prefix}rh_p12_rn_ee_joint" type="fixed">
     <origin xyz="0.0 0.0 0.125" rpy="0 0 0"/>
-    <parent link="rh_p12_rn_base"/>
-    <child link="rh_p12_rn_ee"/>
+    <parent link="${prefix}rh_p12_rn_base"/>
+    <child link="${prefix}rh_p12_rn_ee"/>
   </joint>
   <!-- Gripper end effector link -->
-  <link name="rh_p12_rn_ee">
+  <link name="${prefix}rh_p12_rn_ee">
     <visual>
       <origin xyz="0 0 0" rpy="0 0 0"/>
