Commit message: adjust friction parameters so gripper can grab objects

File: rh_p12_rn_a_description/urdf/rh_p12_rn_a_control.xacro (robot description, xacro)
@@ -7,10 +7,10 @@
         </hardware>
         <joint name="${prefix}rh_r1_joint">
-        <command_interface name="position"/>
-        <state_interface name="position"/>
-        <state_interface name="velocity"/>
-        <state_interface name="effort"/>
-        <state_interface name="torque_enable"/>
-        <state_interface name="hardware_state"/>
+            <command_interface name="position"/>
+            <state_interface name="position"/>
+            <state_interface name="velocity"/>
+            <state_interface name="effort"/>
+            <state_interface name="torque_enable"/>
+            <state_interface name="hardware_state"/>
         </joint>
         <joint name="${prefix}rh_r2">

File: rh_p12_rn_a_description/urdf/rh_p12_rn_a_gripper.xacro (robot description, xacro)
@@ -35,6 +35,6 @@
       <origin xyz="0.0 0.008 0.048" rpy="0 0 0"/>
       <axis xyz="1 0 0"/>
-      <limit velocity="6.5" effort="1000" lower="-0.1" upper="1.1"/>
-      <dynamics damping="0.7"/>
+      <limit velocity="1.0" effort="5" lower="-0.1" upper="1.1"/>
+      <dynamics damping="5.0"/>
     </joint>
     <!-- rh_p12_rn_r1 -->
@@ -67,6 +67,6 @@
       <origin xyz="0.0 0.0493634 0.0285" rpy="0 0 0"/>
       <axis xyz="-1 0 0"/>
-      <limit velocity="6.5" effort="1000" lower="0.0" upper="1.0" />
-      <dynamics damping="0.7"/>
+      <limit velocity="1.0" effort="5" lower="-0.1" upper="1.1" />
+      <dynamics damping="5.0"/>
       <mimic joint="${prefix}rh_r1_joint" multiplier="1"/>
     </joint>
@@ -100,6 +100,6 @@
       <origin xyz="0.0 -0.008 0.048" rpy="0 0 0"/>
       <axis xyz="-1 0 0"/>
-      <limit velocity="6.5" effort="1000" lower="-0.1" upper="1.1" />
-      <dynamics damping="0.7"/>
+      <limit velocity="1.0" effort="5" lower="-0.1" upper="1.1" />
+      <dynamics damping="5.0"/>
       <mimic joint="${prefix}rh_r1_joint" multiplier="1"/>
     </joint>
@@ -133,6 +133,6 @@
       <origin xyz="0.0 -0.0493634 0.0285" rpy="0 0 0"/>
       <axis xyz="1 0 0"/>
-      <limit velocity="6.5" effort="1000" lower="0.0" upper="1.0" />
-      <dynamics damping="0.7"/>
+      <limit velocity="1.0" effort="5" lower="-0.1" upper="1.1" />
+      <dynamics damping="5.0"/>
       <mimic joint="${prefix}rh_r1_joint" multiplier="1"/>
     </joint>
